Commit message: modified some launch files

File: dev_ws/src/midibot_description/urdf/materials.xacro (robot description, xacro)
@@ -4,3 +4,12 @@
   <color rgba="0.700 0.700 0.700 1.000"/>
 </material>
+<material name="black">
+  <color rgba="0.000 0.000 0.000 1.000"/>
+</material>
+<material name="white">
+  <color rgba="1.000 1.000 1.000 1.000"/>
+</material>
+<material name="red">
+  <color rgba="1.000 0.000 0.000 1.000"/>
+</material>
 </robot>

File: dev_ws/src/midibot_description/urdf/midibot.xacro (robot description, xacro)
@@ -4,4 +4,5 @@
 <xacro:include filename="$(find midibot_description)/urdf/midibot.trans" />
 <xacro:include filename="$(find midibot_description)/urdf/midibot.gazebo" />
+<xacro:include filename="$(find midibot_description)/urdf/laser_scan.xacro" />
 <link name="base_link">
   <inertial>
@@ -85,5 +86,5 @@
 </link>
 <joint name="Revolute 1" type="continuous">
-  <origin xyz="-0.090488 -0.436102 0.36973" rpy="0 0 0"/>
+  <origin xyz="-0.152 0.003 -0.043" rpy="0 0 0"/>
   <parent link="base_link"/>
   <child link="back_wheel_1"/>
@@ -91,5 +92,5 @@
 </joint>
 <joint name="Revolute 2" type="continuous">
-  <origin xyz="0.144339 -0.529459 0.36961" rpy="0 0 0"/>
+  <origin xyz="0.083 -0.091 -0.043" rpy="0 0 0"/>
   <parent link="base_link"/>
   <child link="right_wheel_1"/>
@@ -97,5 +98,5 @@
 </joint>
 <joint name="Revolute 3" type="continuous">
-  <origin xyz="0.143827 -0.341455 0.36961" rpy="0 0 0"/>
+  <origin xyz="0.083 0.097 -0.043" rpy="0 0 0"/>
   <parent link="base_link"/>
   <child link="left_wheel_1"/>
